File: projekt_1.kicad_sch (KiCad schematic)
At the start: 33 parts, among them J2 Screw_Terminal_01x03, J3 Conn_WallSocket_Earth, J4 Conn_01x15_Female, J5 Conn_01x15_Female, Q1 BSS138, Q2 BTA16-600C, U2 MOC3041M

Commit message: schematic done
Parts:
- removed C5, C?16V: (no value), symbol Device:C_Polarized_Small
- removed C?: (no value), symbol Device:C
- removed FL1: Choke_Schaffner_RN102-0.3-02-22M, Inductor_THT:Choke_Schaffner_RN102-04-14.0x14.0mm, symbol Filter:Choke_Schaffner_RN102-0.3-02-22M
- removed J3: Conn_WallSocket_Earth, symbol Connector:Conn_WallSocket_Earth
- removed SW?: SW_SPST, symbol Switch:SW_SPST
- added C1, C2, C4: (no value), symbol Device:C_Polarized
- added C2xclass2, C2xclass3: (no value), symbol Device:C
- added FL1: (no value), symbol SSHB21HS-R10300:SSHB21HS-R10300
- added J1, J6: (no value), symbol Connector:Screw_Terminal_01x03
- added J3: (no value), TerminalBlock:TerminalBlock_bornier-3_P5.08mm, symbol Connector:Screw_Terminal_01x03
- added R9: (no value), symbol Device:R
- added SW1: SW_DPST, symbol Switch:SW_DPST
- D1: value Power On Red LED -> (none)
- D2: value WiFi connected - Green LED -> (none)
- D3: renamed from D?; value Heat on LED -> (none)
- D4: renamed from D?; value Empty LED -> (none)
- F3: value 630mA -> (none)
- J2: value Screw_Terminal_01x03 -> (none)
- J4, J5: value Conn_01x15_Female -> (none)
- PS1: value HLK-PM01 -> (none); footprint Converter_ACDC:Converter_ACDC_HiLink_HLK-PMxx -> (none)
- Q1: value BSS138 -> (none); footprint Package_TO_SOT_SMD:SOT-23 -> (none)
- Q2: value BTA16-600C -> (none); footprint Package_TO_SOT_THT:TO-220-3_Vertical -> (none)
- R1: value 220 -> (none)
- R2: value 120 -> (none)
- R3, R5: value 100 -> (none)
- R4: value 10k -> (none)
- R6: value 330 -> (none)
- R7: value 360 -> (none)
- R8: value 39 -> (none)
- RV1: value Varistor -> (none)
- U2: footprint (none) -> Package_DIP:DIP-6_W7.62mm_LongPads
- gave numbers to parts that had none: 3
- renumbered C2 to C2xclass1
Connections:
- net +5V: now also C1.1, C2.1, C4.1, J1.1 (Pin_1), R9.1
- net Earth_Protective: now also C2xclass2.1, C2xclass3.2
- net GND: now also C1.2, C2.2, C4.2, J1.3 (Pin_3)
- net L: now also C2xclass1.1, RV1.1, C2xclass2.2, FL1.1 (N1_1), J6.1 (Pin_1), SW1.4
- net N: now also F2.2, J3.2 (Pin_2), J6.2 (Pin_2), SW1.2
- net OneWire: now also J1.2 (Pin_2), R9.2
- net PE: now also J3.3 (Pin_3)
- net at J2.1 (Pin_1): now also SW1.3
- net at C2xclass1.2, F1.1, RV1.2: now also C2xclass3.1, FL1.2 (N1_2)
- net at C3.2, Q2.1 (A1), R6.2: now also J3.1 (Pin_1)
- net at PS1.1 (AC/L): now also FL1.4 (N2_2)
- net at PS1.2 (AC/N): now also FL1.3 (N2_1)
- net at J2.2 (Pin_2): now also SW1.1; no longer F2.2
Other:
- note added: "137 for 15mA with 3.3V supply"
- note added: "DS18B20 section"
- note added: "Kondensator polipropylenowy"
- note removed: "??"
- note removed: "konfiguracja wyjścia esp jako open-drain"
- moved on the sheet: D3, D4, F1, F2, F3, J2, PS1, R10, R11, R8

Commit message: Add files via upload
Parts:
- removed C2: (no value), symbol Device:C_Polarized
- removed F3: (no value), symbol Device:Fuse
- removed J2: (no value), symbol Connector:Screw_Terminal_01x03
- added H1, H2, H3, H4: MountingHole, MountingHole:MountingHole_3.2mm_M3, symbol Mechanical:MountingHole
- C1: value (none) -> 10u; footprint (none) -> Capacitor_SMD:C_1206_3216Metric_Pad1.33x1.80mm_HandSolder
- C2xclass1, C2xclass2, C2xclass3: value (none) -> 2.2n; footprint (none) -> Capacitor_THT:CP_Axial_L10.0mm_D4.5mm_P15.00mm_Horizontal
- C3: value (none) -> 22n; footprint (none) -> Capacitor_SMD:C_1812_4532Metric_Pad1.57x3.40mm_HandSolder
- C4: value (none) -> 100n; footprint (none) -> Capacitor_SMD:C_1206_3216Metric_Pad1.33x1.80mm_HandSolder
- D1: value (none) -> Power On Red LED; footprint (none) -> LED_THT:LED_D3.0mm
- D2: value (none) -> WiFi connected - Green LED; footprint (none) -> LED_THT:LED_D3.0mm
- D3: value (none) -> Heat on - RED LED; footprint (none) -> LED_THT:LED_D3.0mm
- D4: value (none) -> Empty Orange LED; footprint (none) -> LED_THT:LED_D3.0mm
- F1: value (none) -> Thermal Fuse 72 st.; footprint (none) -> Resistor_THT:R_Axial_DIN0516_L15.5mm_D5.0mm_P30.48mm_Horizontal
- F2: value (none) -> 12.5; footprint (none) -> Fuse:Fuseholder_Cylinder-5x20mm_Stelvio-Kontek_PTF78_Horizontal_Open
- FL1: value (none) -> SSHB21HS-R10300; footprint (none) -> Inductor_THT:SSHB21HSR10300
- J1: value (none) -> Screw_DS18_Terminal_01x03; footprint (none) -> TerminalBlock:TerminalBlock_bornier-3_P5.08mm
- J3: value (none) -> Czajnik_plug
- J4, J5: value (none) -> Conn_01x15_Female; footprint (none) -> Connector_PinHeader_2.54mm:PinHeader_2x15_P2.54mm_Vertical_SMD
- J6: value (none) -> Screw_230v_Terminal_01x03; footprint (none) -> TerminalBlock:TerminalBlock_bornier-3_P5.08mm
- PS1: value (none) -> HLK-PM01; footprint (none) -> Converter_ACDC:Converter_ACDC_HiLink_HLK-PMxx
- Q1: value (none) -> BSS138; footprint (none) -> Package_TO_SOT_SMD:SOT-23
- Q2: value (none) -> BTA16-600C; footprint (none) -> Package_TO_SOT_THT:TO-220-3_Vertical
- R1, R10: value (none) -> 2.2k; footprint (none) -> Resistor_SMD:R_1206_3216Metric_Pad1.30x1.75mm_HandSolder
- R11: value (none) -> 1.2k; footprint (none) -> Resistor_SMD:R_1206_3216Metric_Pad1.30x1.75mm_HandSolder
- R2: value (none) -> 1,2k; footprint (none) -> Resistor_SMD:R_1206_3216Metric_Pad1.30x1.75mm_HandSolder
- R3: value (none) -> 100; footprint (none) -> Resistor_SMD:R_1206_3216Metric_Pad1.30x1.75mm_HandSolder
- R4: value (none) -> 10k; footprint (none) -> Resistor_SMD:R_1206_3216Metric_Pad1.30x1.75mm_HandSolder
- R5: value (none) -> 390; footprint (none) -> Resistor_SMD:R_1206_3216Metric_Pad1.30x1.75mm_HandSolder
- R6: value (none) -> 330; footprint (none) -> Resistor_SMD:R_2512_6332Metric
- R7: value (none) -> 360; footprint (none) -> Resistor_SMD:R_2512_6332Metric
- R8: value (none) -> 39; footprint (none) -> Resistor_SMD:R_2512_6332Metric
- R9: value (none) -> 4.7k; footprint (none) -> Resistor_SMD:R_1206_3216Metric_Pad1.30x1.75mm_HandSolder
- RV1: value (none) -> Varistor; footprint (none) -> Varistor:RV_Disc_D12mm_W3.9mm_P7.5mm
Connections:
- net PE is gone; now on net Earth_Protective: J3.3 (Pin_3)
- net +5V: now also PS1.4 (+Vout)
- net Earth_Protective: now also J6.3 (Pin_3)
- net L: now also C2xclass1.2, C2xclass3.1, F1.1, FL1.2 (N1_2), RV1.2; no longer C2xclass1.1, C2xclass2.2, FL1.1 (N1_1), J6.1 (Pin_1), RV1.1, SW1.4
- net N: now also C2xclass1.1, C2xclass2.2, FL1.1 (N1_1), J6.1 (Pin_1), RV1.1, SW1.4; no longer F2.2, J6.2 (Pin_2), SW1.2
- net 230_L: now reaches SW1.3
- net 230_N: now reaches SW1.1
- new net: F2.2, J6.2 (Pin_2), SW1.2
Other:
- note removed: "137 for 15mA with 3.3V supply"
- note removed: "Kondensator polipropylenowy"
- moved on the sheet: J3
