File: projekt_1.kicad_pcb (KiCad board)
At the start: 2 copper layers, 37 parts, among them J1 Screw_DS18_Terminal_01x03, J2 Screw_230v_Terminal_01x03, J3 Czajnik_plug, J4 Conn_01x15_Female, J5 Conn_01x15_Female, J6 Screw_230v_Terminal_01x03, Q1 BSS138, Q2 BTA16-600C, U2 MOC3041M

Commit message: Add files via upload
Parts:
- removed C2: 1u, Capacitor_SMD:CP_Elec_4x5.3
- removed F3: 630mA, Fuse:Fuseholder_Cylinder-5x20mm_Stelvio-Kontek_PTF78_Horizontal_Open
- removed J2: Screw_230v_Terminal_01x03, TerminalBlock:TerminalBlock_bornier-3_P5.08mm
- added H1: MountingHole, MountingHole:MountingHole_3.2mm_M3, F.Cu at (26.9, 17.4)
- added H2: MountingHole, MountingHole:MountingHole_3.2mm_M3, F.Cu at (119.4, 17.8)
- added H3: MountingHole, MountingHole:MountingHole_3.2mm_M3, F.Cu at (119.4, 101.6)
- added H4: MountingHole, MountingHole:MountingHole_3.2mm_M3, F.Cu at (26.9, 101.2)
- C1, C4: footprint Capacitor_SMD:CP_Elec_4x5.3 -> Capacitor_SMD:C_1206_3216Metric_Pad1.33x1.80mm_HandSolder
- C3: footprint Capacitor_THT:CP_Axial_L10.0mm_D6.0mm_P15.00mm_Horizontal -> Capacitor_SMD:C_1812_4532Metric_Pad1.57x3.40mm_HandSolder
- F2: value 200mA -> 12.5
- J4, J5: footprint Connector_PinHeader_2.54mm:PinHeader_2x15_P2.54mm_Vertical -> Connector_PinHeader_2.54mm:PinHeader_2x15_P2.54mm_Vertical_SMD
- R1, R10, R11, R2, R3, R4, R5, R9: footprint Resistor_SMD:R_0603_1608Metric -> Resistor_SMD:R_1206_3216Metric_Pad1.30x1.75mm_HandSolder
- U2: footprint Package_DIP:DIP-6_W7.62mm_LongPads -> Package_DIP:DIP-6_W8.89mm_SMDSocket_LongPads
- moved R8 172.4 mm to (27.9, 84.7)
- moved J3 164.7 mm to (37.1, 95.5)
- moved C2xclass2 162.2 mm to (43.8, 52.0), turned to 180 degrees
- moved J6 152.3 mm to (45.9, 23.5), turned to -90 degrees
- moved C2xclass3 150.0 mm to (29.1, 59.0)
- moved C3 144.7 mm to (35.5, 84.8)
- moved C4 144.7 mm to (77.7, 100.5), turned to -90 degrees
- moved Q2 143.2 mm to (36.0, 72.3), turned to 0 degrees
- moved C1 139.6 mm to (81.3, 100.5), turned to -90 degrees
- moved F2 110.4 mm to (72.3, 49.7), turned to 180 degrees
- moved C2xclass1 109.2 mm to (55.6, 21.9), turned to -90 degrees
- moved PS1 106.3 mm to (104.1, 21.0), turned to -90 degrees
- moved FL1 74.9 mm to (63.5, 21.9)
- moved R6 68.4 mm to (43.2, 84.7), turned to 180 degrees
- moved J5 67.6 mm to (103.1, 80.2)
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Connections:
- C2xclass1 pad 1: /L -> /N
- C2xclass1 pad 2: Net-(C2xclass1-Pad2) -> /L
- C2xclass2 pad 2: /L -> /N
- C2xclass3 pad 1: Net-(C2xclass1-Pad2) -> /L
- F1 pad 1: Net-(C2xclass1-Pad2) -> /L
- F2 pad 2: /N -> Net-(F2-Pad2)
- FL1 pad 1: /L -> /N
- FL1 pad 2: Net-(C2xclass1-Pad2) -> /L
- FL1 pad 3: Net-(PS1-Pad2) -> Net-(FL1-Pad3)
- FL1 pad 4: Net-(PS1-Pad1) -> Net-(FL1-Pad4)
- J3 pad 3: /PE -> Earth_Protective
- J4 pad 1: (no net) -> +3V3
- J4 pad 10: (no net) -> /D27
- J4 pad 11: (no net) -> /D14
- J4 pad 12: (no net) -> /D12
- J4 pad 13: (no net) -> /D13
- J4 pad 14: (no net) -> GND
- J4 pad 15: (no net) -> +5V
- J4 pad 2: (no net) -> /VP
- J4 pad 3: (no net) -> /VN
- J4 pad 4: (no net) -> /D34
- J4 pad 5: (no net) -> /D35
- J4 pad 6: (no net) -> /D32
- J4 pad 7: (no net) -> /D33
- J4 pad 8: (no net) -> /D25
- J4 pad 9: (no net) -> /D26
- J5 pad 14: /D22 -> /D18?
- J5 pad 16: (no net) -> /Empty
- J5 pad 18: (no net) -> /TX2
- J5 pad 2: GND -> /D23
- J5 pad 20: (no net) -> /RX2
- J5 pad 22: (no net) -> /OneWire
- J5 pad 24: (no net) -> /Triac
- J5 pad 26: (no net) -> /WiFi_LED
- J5 pad 6: /RX2 -> /TX0
- J5 pad 8: /Empty -> /RX0
- J6 pad 1: /L -> /N
- J6 pad 2: /N -> Net-(F2-Pad2)
- PS1 pad 1: Net-(PS1-Pad1) -> Net-(FL1-Pad3)
- PS1 pad 2: Net-(PS1-Pad2) -> Net-(FL1-Pad4)
- PS1 pad 4: Net-(F3-Pad2) -> +5V
- RV1 pad 1: /L -> /N
- RV1 pad 2: Net-(C2xclass1-Pad2) -> /L
Routing:
- net /L: track 0.00 -> 176.6 mm
- net +5V: track 0.00 -> 135.3 mm
- net /N: track 0.00 -> 110.7 mm
- net /Drain: track 0.00 -> 86.3 mm, vias 0 -> 2
- net Earth_Protective: track 0.00 -> 67.7 mm
- net Net-(R5-Pad1): track 0.00 -> 50.9 mm, vias 0 -> 2
- net /OneWire: track 0.00 -> 43.0 mm, vias 0 -> 1
- net Net-(FL1-Pad3): track 0.00 -> 30.9 mm
- net Net-(Q2-Pad3): track 0.00 -> 27.7 mm
- net Net-(C3-Pad2): track 0.00 -> 26.5 mm
- net Net-(F2-Pad2): track 0.00 -> 22.8 mm
- net Net-(F1-Pad2): track 0.00 -> 17.8 mm
- net Net-(FL1-Pad4): track 0.00 -> 15.0 mm
- net /Triac: track 0.00 -> 14.4 mm
- net /Empty: track 0.00 -> 13.9 mm
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- added copper zone on B.Cu, net GND
- added copper zone on F.Cu, net GND
Other:
- board outline added: 99.6 x 91.3 mm
- board text added: "SMARTCZAJNIK ver.1.0"

Commit message: Add files via upload
Parts:
- moved H4 0.25 mm to (26.9, 101.0)
- moved H3 0.13 mm to (119.4, 101.5)
Other:
- board size 99.6 x 91.3 mm -> 99.8 x 90.7 mm
Changed lines of the file:
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@@
       (drillshape 0)
       (scaleselection 1)
-      (outputdirectory "../../../Desktop/smartczajnik/pdfy_gerbery/")
+      (outputdirectory "gerber/")
     )
   )
@@
   )
   (footprint "MountingHole:MountingHole_3.2mm_M3" (layer "F.Cu")
-    (at 26.8986 101.2192)
+    (at 26.8986 100.9652)
     (descr "Mounting Hole 3.2mm, no annular, M3")
     (tags "mounting hole 3.2mm no annular m3")
@@
   )
   (footprint "MountingHole:MountingHole_3.2mm_M3" (layer "F.Cu")
-    (at 119.38 101.6)
+    (at 119.38 101.4732)
     (descr "Mounting Hole 3.2mm, no annular, M3")
     (tags "mounting hole 3.2mm no annular m3")
@@
     )
   )
-  (gr_line (start 23.3426 104.7752) (end 23.3426 13.8432) (layer "Edge.Cuts") (width 0.2))
-  (gr_line (start 122.936 105.156) (end 23.3426 104.7752) (layer "Edge.Cuts") (width 0.2))
-  (gr_line (start 23.3426 13.8432) (end 122.936 14.224) (layer "Edge.Cuts") (width 0.2))
-  (gr_line (start 122.936 14.224) (end 122.936 105.156) (layer "Edge.Cuts") (width 0.2))
+  (gr_rect (start 123.1646 13.8432) (end 23.3426 104.5212) (layer "Edge.Cuts") (width 0.1) (fill none))
   (gr_text "SMARTCZAJNIK ver.1.0" (at 39.8526 15.5196) (layer "F.SilkS")
     (effects (font (size 1 1) (thickness 0.15)))
